File: ecad/ds3231_breakout/ds3231_breakout.sch (EAGLE design)
At the start: 6 parts, among them IC1 DS3231, J1 PTH RA MALE

Commit message: Create DS3231 breakout vesion.  Updated libraries.
Parts:
- BATT1: device _batteries:BATTERY_COIN-CELL_SMD_3V_20MM -> _batteries:BATTERY_COIN-CELL_PTH_3V_20MM
Changed lines of the file:
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@@
 <part name="SUPPLY7" library="_power_symbols" deviceset="3V" device=""/>
 <part name="SUPPLY8" library="_power_symbols" deviceset="GND" device=""/>
-<part name="BATT1" library="_batteries" deviceset="BATTERY_COIN-CELL" device="_SMD_3V_20MM" package3d_urn="urn:adsk.eagle:package:2959529/4" value="CR2032 225mAh/3V"/>
 <part name="IC1" library="_special" deviceset="DS3231" device="_DS3231_RTC_CLK_I2C_SOIC-16" package3d_urn="urn:adsk.eagle:package:7208538/1" value="DS3231"/>
 <part name="J1" library="_connectors" deviceset="1X06" device="PTH_RA_MALE_2.54MM" package3d_urn="urn:adsk.eagle:package:7208728/1" value="PTH RA MALE"/>
 <part name="SUPPLY9" library="_power_symbols" deviceset="VCC" device=""/>
 <part name="SUPPLY10" library="_power_symbols" deviceset="GND" device=""/>
+<part name="BATT1" library="_batteries" deviceset="BATTERY_COIN-CELL" device="_PTH_3V_20MM" package3d_urn="urn:adsk.eagle:package:4291813/3" value="CR2032 225mAh/3V"/>
 </parts>
 <sheets>
@@
 <instance part="SUPPLY7" gate="G$1" x="15.24" y="48.26" smashed="yes"/>
 <instance part="SUPPLY8" gate="GND" x="15.24" y="27.94" smashed="yes"/>
-<instance part="BATT1" gate="G$1" x="15.24" y="40.64" smashed="yes">
-<attribute name="NAME" x="15.494" y="41.148" size="1.27" layer="95" font="vector" ratio="10"/>
-<attribute name="VALUE" x="15.494" y="38.862" size="0.635" layer="96" font="vector" ratio="10" align="top-left"/>
-</instance>
 <instance part="IC1" gate="G$1" x="50.8" y="40.64" smashed="yes">
 <attribute name="NAME" x="50.8" y="48.514" size="1.27" layer="95" font="vector" ratio="10" align="bottom-center"/>
@@
 <instance part="SUPPLY9" gate="VCC" x="114.3" y="38.1" smashed="yes"/>
 <instance part="SUPPLY10" gate="GND" x="104.14" y="27.94" smashed="yes"/>
+<instance part="BATT1" gate="G$1" x="15.24" y="40.64" smashed="yes">
+<attribute name="NAME" x="15.494" y="41.148" size="1.27" layer="95" font="vector" ratio="10"/>
+<attribute name="VALUE" x="15.494" y="38.862" size="0.635" layer="96" font="vector" ratio="10" align="top-left"/>
+</instance>
 </instances>
 <busses>
